File: fafnir/fafnir.sch (KiCad schematic (older format))
At the start: 16 parts, among them IC1 CD4049UBE

Commit message: v2 schematic, with Baxandall tone stack
Parts:
- added BASS1, TREBLE1: 100kA, potentiometers:16MM_T.MOUNT, symbol Device:R_POT_US
- added C12, C15: 22nF, caps-film:0.2_.SML, symbol Device:C_Small
- added C13: 47nF, caps-film:0.2_.SML, symbol Device:C_Small
- added C14: 2.2nF, caps-film:0.2_.SML, symbol Device:C_Small
- added C8: 47uF, caps-elec:050.FLAT, symbol Device:CP1
- added C?: 4.7uF, symbol Device:CP1_Small
- added R12: 15k, resistors:0.2_, symbol Device:R_US
- added R13: 10k, resistors:0.2_, symbol Device:R_US
- added R14: 12k, resistors:0.2_, symbol Device:R_US
- added R15: 4.7k, resistors:0.2_, symbol Device:R_US
- added R5, R9: 100k, resistors:0.2_, symbol Device:R_US
- added U?: LF411, symbol LF411:LF411_A
Connections:
- net labels added: VA
- wire segments 51 -> 86
Other:
- moved on the sheet: C1, C2, C3, C4, C5, C6, C7, D1, GAIN1, IC1, R1, R2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
